Commit message: feat: picknik_006_gen3 hardware config (Robotiq 2F-85 + wrist RealSense)
Asset-ID branch for the specific Kinova Gen3 7DoF + Robotiq 2F-85 + wrist
RealSense D415 setup. Follows the doc's "per-physical-robot
customization" naming convention
(docs.picknik.ai/how_to/configuration_tutorials/robot_and_objective_inheritance/#robot-naming-conventions):
new asset-ID branches fork main (which carries the bare-arm boilerplate
kinova_gen3_{mock,sim,hw}) and rename their configs with the asset-ID
prefix.

Inheritance chain (doc-canonical mock -> sim -> hw)
---------------------------------------------------
    picknik_006_gen3_mock  (trunk; no based_on_package)
       |
       +--> picknik_006_gen3_sim   based_on_package: picknik_006_gen3_mock
       |                           overrides urdf_params to drop the
       |                           gripper + wrist RealSense so the URDF
       |                           matches the bare-arm MuJoCo scene.xml
       |                           inherited from main.
       |
       +--> picknik_006_gen3_hw    based_on_package: picknik_006_gen3_sim
                                   restores gripper + wrist_realsense
                                   urdf_params, sets real-hardware fields
                                   (simulated: False, robot_ip,
                                   use_fake_hardware: false), re-adds
                                   robotiq_gripper_controller and
                                   fault_controller, uncomments the
                                   cameras.launch.xml include.

Renames
-------
* kinova_gen3_mock  -> picknik_006_gen3_mock
* kinova_gen3_sim   -> picknik_006_gen3_sim
* kinova_gen3_hw    -> picknik_006_gen3_hw
  (kinova_pstop_manager keeps its name -- helper library, not a robot
  config, so the asset-ID prefix does not apply per the doc.)

picknik_006_gen3_mock (trunk additions over main's kinova_gen3_mock)
--------------------------------------------------------------------
* description/picknik_kinova_gen3.xacro: restore from main's pre-restructure
  history -- gripper-conditional load, wrist_realsense xacro:if block,
  Robotiq-parented grasp_link / finger_tip_closed_point.
* description/kortex_robot.xacro: restore the <xacro:unless "${not gripper}">
  load_gripper block that includes robotiq_2f_85_macro.xacro.
* description/robotiq_2f_85_gripper.urdf, robotiq_2f_85_macro.xacro:
  restored from pre-restructure history (the trimmed-on-main Robotiq URDF
  + macros).
* config/moveit/picknik_kinova_gen3_base.srdf: restored full SRDF
  (gripper group, open/closed group_states, robotiq + wrist-camera
  disable_collisions pairs).
* config/control/picknik_kinova_gen3.ros2_control.yaml: restore
  robotiq_gripper_controller and fault_controller plus the bottom-of-file
  robotiq_gripper_controller parameter block.
* config/config.yaml urdf_params: add gripper, gripper_joint_name,
  use_internal_bus_gripper_comm, wrist_realsense.
* config/config.yaml controllers_active_at_startup: add
  robotiq_gripper_controller.
* package.xml: add realsense2_description, robotiq_description exec_depends.

picknik_006_gen3_sim (slim override over _mock)
------------------------------------------------
* config/config.yaml: override urdf_params to set gripper="" and
  wrist_realsense="false" so the URDF reverts to bare-arm matching the
  inherited MuJoCo scene.
* config/config.yaml: override controllers_active_at_startup to drop
  robotiq_gripper_controller (no gripper to drive in sim).
* description/mujoco/scene.xml: unchanged (bare-arm scene from main).

picknik_006_gen3_hw (slim override over _sim)
----------------------------------------------
* config/config.yaml: re-enable gripper + wrist_realsense urdf_params for
  the real arm. Add real-hardware fields (simulated: False, robot_ip,
  use_fake_hardware: false). Add fault_controller +
  robotiq_gripper_controller to controllers_active_at_startup.
* launch/agent_bridge.launch.xml: uncomment the cameras.launch.xml include
  (was the existing "Uncomment for kinovas with embedded realsense wrist
  camera" line).
* package.xml: add realsense2_camera (runtime D415 driver) exec_depend.

Top-level
---------
* README.md rewritten for this branch: describes the asset-ID convention,
  the inheritance chain, and clarifies that the branch does not merge
  back into main.
* .gitmodules unchanged -- internal-bus Robotiq + integrated Vision Module
  works with the existing ros2_kortex / ros2_kortex_vision /
  picknik_accessories submodules.

Verification (after pushing and pulling submodules)
---------------------------------------------------
1. colcon build --packages-select picknik_006_gen3_hw picknik_006_gen3_sim
   picknik_006_gen3_mock
2. xacro $(ros2 pkg prefix picknik_006_gen3_mock --share)/description/
   picknik_kinova_gen3.xacro gripper:=robotiq_2f_85 wrist_realsense:=true |
   check_urdf -
3. moveit_pro run -c picknik_006_gen3_mock  (gripper drivable via fake hw)
4. moveit_pro run -c picknik_006_gen3_sim   (bare-arm MuJoCo, motion-only)
5. With arm + RealSense attached:
   moveit_pro run -c picknik_006_gen3_hw    (full kit live)

File: src/picknik_006_gen3_mock/description/kortex_robot.xacro (robot description, xacro)
@@ -6,4 +6,6 @@
     prefix
     arm
+    gripper
+    gripper_joint_name
     dof
     vision
@@ -15,4 +17,5 @@
     session_inactivity_timeout_ms
     connection_inactivity_timeout_ms
+    use_internal_bus_gripper_comm:=false
     use_fake_hardware:=false
     fake_sensor_commands:=false
@@ -24,9 +27,7 @@
     use_external_cable:=false
     initial_positions:=${dict(joint_1=0.0,joint_2=0.0,joint_3=0.0,joint_4=0.0,joint_5=0.0,joint_6=0.0,joint_7=0.0)}
-    gripper:=
-    gripper_joint_name:=
-    use_internal_bus_gripper_comm:=false
     gripper_max_velocity:=100.0
     gripper_max_force:=100.0
+    gripper_com_port:=/dev/ttyUSB0
     moveit_active:=false">
     <!-- Include and load arm macro files -->
@@ -58,14 +59,31 @@
       <xacro:insert_block name="origin" />
     </xacro:load_arm>
-    <!-- Boilerplate has no gripper; expose tool_frame at the wrist. Branches
-         that add a gripper override gripper / gripper_joint_name and bring in
-         their own gripper xacro to override this section. -->
-    <link name="${prefix}tool_frame"/>
-    <joint name="${prefix}tool_frame_joint" type="fixed">
-      <origin xyz="0 0 0" rpy="0 0 0" />
-      <parent link="${prefix}${last_arm_link}" />
-      <child link="${prefix}tool_frame" />
-      <axis xyz="0 0 0" />
-    </joint>
+    <!-- If no gripper, define tool frame here -->
+    <xacro:if value="${not gripper}">
+      <link name="${prefix}tool_frame"/>
+      <joint name="${prefix}tool_frame_joint" type="fixed">
+        <origin xyz="0 0 0" rpy="0 0 0" />
+        <parent link="${prefix}${last_arm_link}" />
+        <child link="${prefix}tool_frame" />
+        <axis xyz="0 0 0" />
+      </joint>
+    </xacro:if>
+    <!-- Include and load the gripper if defined -->
+    <xacro:unless value="${not gripper}">
+      <xacro:include filename="$(find picknik_006_gen3_mock)/description/robotiq_2f_85_macro.xacro" />
+      <!-- last_arm_link is defined in "$(find kortex_description)/arms/${arm}/urdf/${arm}_macro.xacro" -->
+      <xacro:load_gripper
+        parent="${prefix}${last_arm_link}"
+        prefix="${prefix}"
+        use_fake_hardware="${use_fake_hardware}"
+        fake_sensor_commands="${fake_sensor_commands}"
+        sim_ignition="${sim_ignition}"
+        sim_isaac="${sim_isaac}"
+        isaac_joint_commands="${isaac_joint_commands}"
+        isaac_joint_states="${isaac_joint_states}"
+        com_port="${gripper_com_port}"
+        use_internal_bus_gripper_comm="${use_internal_bus_gripper_comm}"
+        moveit_active="${moveit_active}"/>
+    </xacro:unless>
   </xacro:macro>
 </robot>

Commit message: fix(kortex_robot.xacro): call robotiq_gripper directly, bypass kortex's broken load_gripper
kortex_description's load_gripper intermediate macro
(grippers/robotiq_2f_85/urdf/robotiq_2f_85_macro.xacro at our pinned
732b96f9) didn't finish the sim_ignition -> sim_gazebo rename: it accepts
sim_gazebo from the outer call but still forwards the value under the
legacy param name sim_ignition to the inner robotiq_gripper macro.

    <xacro:robotiq_gripper
        ...
        sim_ignition="${sim_gazebo}"  <-- legacy name
        ...

The current ros2_robotiq_gripper version we pin (12e6232) renamed the
inner macro's param to sim_gazebo and dropped sim_ignition. So URDF
generation fails with:

    Invalid parameter "sim_ignition"
    when instantiating macro: robotiq_gripper
                              (robotiq_description/urdf/robotiq_2f_85_macro.urdf.xacro)

We can't fix the kortex_description submodule from this workspace, so
skip the broken intermediate and call robotiq_gripper directly from our
kortex_robot.xacro. The include_ros2_control logic mirrors what
kortex_description's load_gripper computed.

Side effects:
* Drops the moveit_active flag — robotiq_gripper doesn't accept it
  anyway (kortex's load_gripper was the only consumer).
* The include filename is now parameterised by ${gripper}, so this also
  works for robotiq_2f_140 if a downstream branch switches the gripper.

Same fix needed on picknik_006_gen3-quest-teleop via the usual rebase.

File: src/picknik_006_gen3_mock/description/kortex_robot.xacro (robot description, xacro)
@@ -69,13 +69,26 @@
       </joint>
     </xacro:if>
-    <!-- Include and load the gripper if defined -->
+    <!-- Include and load the gripper if defined.
+         We bypass kortex_description's intermediate `load_gripper` macro
+         because it forwards sim_gazebo to the inner robotiq_gripper under
+         the LEGACY param name sim_ignition, which the current
+         robotiq_description macro no longer accepts. Call robotiq_gripper
+         directly with the right param name. -->
     <xacro:unless value="${not gripper}">
-      <xacro:include filename="$(find kortex_description)/grippers/robotiq_2f_85/urdf/robotiq_2f_85_macro.xacro" />
+      <xacro:include filename="$(find robotiq_description)/urdf/${gripper}_macro.urdf.xacro" />
+      <!-- ros2_control is needed when not using the Kinova internal bus, or
+           when running mock/MuJoCo/Isaac. Logic mirrors kortex_description's
+           load_gripper. -->
+      <xacro:property name="include_ros2_control" value="false"/>
+      <xacro:if value="${sim_gazebo or sim_isaac or use_fake_hardware or not use_internal_bus_gripper_comm}">
+        <xacro:property name="include_ros2_control" value="true"/>
+      </xacro:if>
       <!-- last_arm_link is defined in "$(find kortex_description)/arms/${arm}/urdf/${arm}_macro.xacro" -->
-      <xacro:load_gripper
+      <xacro:robotiq_gripper
+        name="RobotiqGripperHardwareInterface"
         parent="${prefix}${last_arm_link}"
         prefix="${prefix}"
         use_fake_hardware="${use_fake_hardware}"
-        fake_sensor_commands="${fake_sensor_commands}"
+        mock_sensor_commands="${fake_sensor_commands}"
         sim_gazebo="${sim_gazebo}"
         sim_isaac="${sim_isaac}"
@@ -84,5 +97,7 @@
         com_port="${gripper_com_port}"
         use_internal_bus_gripper_comm="${use_internal_bus_gripper_comm}"
-        moveit_active="${moveit_active}"/>
+        include_ros2_control="${include_ros2_control}">
+        <origin xyz="0 0 0" rpy="0 0 0"/>
+      </xacro:robotiq_gripper>
     </xacro:unless>
   </xacro:macro>

Commit message: fix: re-pin ros2_robotiq_gripper to humble branch (e78b482) for parity with UR _hw
Previously pinned to ros2_robotiq_gripper main (12e6232), which carried
PR #54 renaming the inner robotiq_gripper macro's `sim_ignition` param
to `sim_gazebo`. That rename never made it to the humble branch and
kortex_description (our pinned 732b96f9) still forwards sim_ignition
under the legacy name, so the kortex->robotiq layer failed with
"Invalid parameter sim_ignition".

Working around that required bypassing kortex_description's
load_gripper intermediate macro and calling robotiq_gripper directly
(commit 502aaff). That's an extra local patch to maintain.

Switch to the humble branch tip (e78b482) instead. The humble branch
cherry-picks the substantive fixes from main:

  93ecde7 Replace fake_sensor_commands with mock_sensor_commands (#62)
  e5656b1 Fix gripper speed and force parameter init (#83)
  c652540 Add com_port launch & xacro arguments (#78)
  2ff8545 update urdf mesh filenames to use package path (#68)

...but deliberately omits #54 (the sim_ignition->sim_gazebo rename),
so it pairs cleanly with our older kortex_description without any
local bypass. moveit_pro_ur_ws's robotiq-bearing configs use the same
e78b482 pin, so we match the convention.

Trade-off: humble lacks two main-only commits we'd otherwise want:

  12e6232 Include <algorithm> to avoid compiler issues (#82)
  856753c Fix ResourceManager parameters on humble (#74)

The first is a portability nit (only matters on toolchains whose
<vector>/<array> headers don't transitively include <algorithm>); the
Pro humble base image's gcc 11 doesn't trip on it. The second is a
ResourceManager param fix that humble apparently doesn't need (UR _hw
configs build fine without it).

Reverts commit 502aaff (bypass-load_gripper) since the bypass is no
longer needed -- kortex_description's load_gripper macro pairs cleanly
with the humble branch's robotiq_gripper signature.

File: src/picknik_006_gen3_mock/description/kortex_robot.xacro (robot description, xacro)
@@ -69,26 +69,13 @@
       </joint>
     </xacro:if>
-    <!-- Include and load the gripper if defined.
-         We bypass kortex_description's intermediate `load_gripper` macro
-         because it forwards sim_gazebo to the inner robotiq_gripper under
-         the LEGACY param name sim_ignition, which the current
-         robotiq_description macro no longer accepts. Call robotiq_gripper
-         directly with the right param name. -->
+    <!-- Include and load the gripper if defined -->
     <xacro:unless value="${not gripper}">
-      <xacro:include filename="$(find robotiq_description)/urdf/${gripper}_macro.urdf.xacro" />
-      <!-- ros2_control is needed when not using the Kinova internal bus, or
-           when running mock/MuJoCo/Isaac. Logic mirrors kortex_description's
-           load_gripper. -->
-      <xacro:property name="include_ros2_control" value="false"/>
-      <xacro:if value="${sim_gazebo or sim_isaac or use_fake_hardware or not use_internal_bus_gripper_comm}">
-        <xacro:property name="include_ros2_control" value="true"/>
-      </xacro:if>
+      <xacro:include filename="$(find kortex_description)/grippers/robotiq_2f_85/urdf/robotiq_2f_85_macro.xacro" />
       <!-- last_arm_link is defined in "$(find kortex_description)/arms/${arm}/urdf/${arm}_macro.xacro" -->
-      <xacro:robotiq_gripper
-        name="RobotiqGripperHardwareInterface"
+      <xacro:load_gripper
         parent="${prefix}${last_arm_link}"
         prefix="${prefix}"
         use_fake_hardware="${use_fake_hardware}"
-        mock_sensor_commands="${fake_sensor_commands}"
+        fake_sensor_commands="${fake_sensor_commands}"
         sim_gazebo="${sim_gazebo}"
         sim_isaac="${sim_isaac}"
@@ -97,7 +84,5 @@
         com_port="${gripper_com_port}"
         use_internal_bus_gripper_comm="${use_internal_bus_gripper_comm}"
-        include_ros2_control="${include_ros2_control}">
-        <origin xyz="0 0 0" rpy="0 0 0"/>
-      </xacro:robotiq_gripper>
+        moveit_active="${moveit_active}"/>
     </xacro:unless>
   </xacro:macro>
