Commit message: fix: repair the Kinova boilerplate so its configs can launch
No configuration in this workspace could start. Repairs, each verified
against picknikciuser/moveit-pro:main-jazzy:

URDF generation was impossible. kortex_robot.xacro declared `gripper:=`
and `gripper_joint_name:=` with no default values, so xacro consumed the
next token as gripper's default and gripper_joint_name was never declared
— every invocation failed with `Invalid parameter
"gripper_joint_name"`. Give both an explicit empty default.

kinova_gen3_hw and kinova_gen3_sim each named a robot_drivers_to_persist
launch file absent from their own package, and the Agent resolves those
with a plain path join and no fallback search, so both raised at bringup.
Drop the overrides so they inherit kinova_gen3_mock's. Delete the 0-byte
kinova_gen3_hw/launch/bringup.launch.py. Re-parent kinova_gen3_hw onto
kinova_gen3_mock directly rather than routing through the simulator config
to reach it.

Three controllers were listed in controllers_inactive_at_startup with no
parameter blocks, so they could not load. Add them. Delete
twist_controller, which no startup list named and whose `tcp` command
interface only the Kortex hardware exports, so it could never load under
the mock hardware this shared manifest also serves. Delete the two
unreferenced per-package manifests, which configured a gripper joint and
an fts/fts_link sensor the bare-arm URDF does not define.

kinova_gen3_hw came up permanently faulted once its driver launch worked.
protective_stop_manager_node watchdogs /fault_controller/internal_fault,
which nothing published on hardware because no manifest declared a
fault_controller; mock gets it from mock_kinova_client_node instead.
Declare fault_controller in the shared manifest, activate it from
kinova_gen3_hw only, and give the watchdog a bounded startup grace period
measured on a steady clock — the Agent starts this node before the
controller manager, so some grace is always needed, but waiting
indefinitely for a first message would report NORMAL forever if the
controller never activated.

Motion limits did not match the arm. Acceleration was 1.0 rad/s^2 on
joints 1-4 and 10.0 on joints 5-7, matching nothing in ros2_kortex, which
ships 8.6 uniformly for the Gen3 7DoF. stop_accelerations sat below the
accelerations it must arrest, so an abort decelerated more slowly than the
motion it was aborting. default_path_tolerance was 0.5 rad — roughly 29
degrees of tracking error before abort — carried over from a zero-gravity
satellite demo. Set 8.6, 30.0 and 0.05 respectively.

The gripper recipe the README documented did nothing:
picknik_kinova_gen3.xacro declared no xacro:arg for gripper,
gripper_joint_name or use_internal_bus_gripper_comm and hardcoded all
three. Declare and forward them, and rewrite the documentation to state
what they actually achieve — the Kortex hardware param and the
ros2_control joint, but no links and no kinematic joint — so a complete
overlay needs a gripper description, a controller and an SRDF group too.

Also: delete kinova_gen3_hw's objectives and waypoints, which the Agent
never loaded because the config did not override those keys; delete
cameras.yaml, which declared two RealSense D415s this arm does not have;
remove phantom gripper joints from both joint_limits.yaml files; drop hw's
pose_jog and joint_jog, byte-identical to mock's; give mock's robot_ip a
non-empty placeholder, since merge matches inherited list entries by
truthiness and a falsy value makes a child's override append rather than
replace; lower the table so its top clears base_link by more than the
collision padding; document the Kortex factory-default credentials, which
reach /robot_description on the hardware path; declare MOVEIT_DOCKER_TAG
and MOVEIT_ROS_DISTRO so --build-arg is not silently ignored; and move to
the picknikciuser/moveit-pro Jazzy base image with package versions at
10.0.0.

kinova_gen3_sim is left non-functional and documented as such. It fails at
URDF generation because the `%>>` syntax on its use_fake_hardware was
removed in MoveIt Pro 6.0.0, and it could not run MuJoCo regardless: no
<ros2_control> block selects the MujocoSystem plugin, which needs a change
to the pinned ros2_kortex to arrange.

Adds test_config_references.py, which resolves the based_on_package chain
with the product's own merge and asserts that referenced files exist, that
startup controllers have a type and parameters, that no controller is
declared but never loaded, that no urdf_params key resolves twice, that
kinova_gen3_hw activates fault_controller, and that every config package
ships a non-empty agent_bridge.launch.xml. It fails 5 tests against the
tree before this change.

Verified: rosdep install exit 0, colcon build exit 0 for all 11 packages,
colcon test 30 tests 0 failures, both bare-arm URDFs generate with the
correct hardware plugin per config and no stray camera or gripper links.
Nothing here is hardware-tested — no Kinova arm was available. The
stop_accelerations change in particular wants a cancel-during-motion test
on a real arm.

File: src/kinova_gen3_mock/description/kortex_robot.xacro (robot description, xacro)
@@ -24,6 +24,6 @@
     use_external_cable:=false
     initial_positions:=${dict(joint_1=0.0,joint_2=0.0,joint_3=0.0,joint_4=0.0,joint_5=0.0,joint_6=0.0,joint_7=0.0)}
-    gripper:=
-    gripper_joint_name:=
+    gripper:=''
+    gripper_joint_name:=''
     use_internal_bus_gripper_comm:=false
     gripper_max_velocity:=100.0

File: src/kinova_gen3_mock/description/picknik_kinova_gen3.xacro (robot description, xacro)
@@ -21,4 +21,19 @@
     <xacro:arg name="isaac_joint_states" default="/isaac_joint_states" />
     <xacro:arg name="use_external_cable" default="false" />
+    <!-- Gripper selection, forwarded to ros2_kortex's load_arm. The boilerplate
+         mounts no gripper, so these default to empty and tool_frame stays at the
+         wrist flange.
+         WARNING: setting these alone does NOT mount a gripper. load_arm uses them
+         for the Kortex hardware block and to add the gripper joint to
+         <ros2_control>, but contributes no links and no kinematic joint, so a
+         config that sets only these produces a model whose <ros2_control> block
+         references a joint the kinematic model does not contain. A complete
+         gripper overlay also needs a gripper description include, a gripper
+         controller in the ros2_control manifest, and a gripper group in the SRDF.
+         See "Adding a Robotiq gripper" in the workspace README, and the
+         picknik_006_gen3 branch for a reference implementation. -->
+    <xacro:arg name="gripper" default="" />
+    <xacro:arg name="gripper_joint_name" default="" />
+    <xacro:arg name="use_internal_bus_gripper_comm" default="false" />
     <!-- Simulator-specific args (no-ops for mock and hw; consumed by inheriting
          configs that select a MuJoCo or Isaac scene). -->
@@ -36,12 +51,12 @@
     <!-- convert to property to use substitution in function -->
     <xacro:property name="initial_positions_file" default="$(arg initial_positions_file)"/>
-    <!-- Load the robot. No gripper is mounted in this boilerplate config; the
-         Kinova-integrated wrist Vision Module is enabled via vision="true". -->
+    <!-- Load the robot. No gripper is mounted by default; the Kinova-integrated
+         wrist Vision Module is enabled via vision="true". -->
     <xacro:load_robot
       parent="world"
       prefix="$(arg prefix)"
       arm="$(arg arm)"
-      gripper=""
-      gripper_joint_name=""
+      gripper="$(arg gripper)"
+      gripper_joint_name="$(arg gripper_joint_name)"
       dof="$(arg dof)"
       vision="$(arg vision)"
@@ -53,5 +68,5 @@
       session_inactivity_timeout_ms="$(arg session_inactivity_timeout_ms)"
       connection_inactivity_timeout_ms="$(arg connection_inactivity_timeout_ms)"
-      use_internal_bus_gripper_comm="false"
+      use_internal_bus_gripper_comm="$(arg use_internal_bus_gripper_comm)"
       use_fake_hardware="$(arg use_fake_hardware)"
       fake_sensor_commands="$(arg fake_sensor_commands)"
@@ -64,6 +79,10 @@
     </xacro:load_robot>
     <!-- Environment -->
+    <!-- The table top must stay clear of base_link by more than the collision
+         padding applied to both, or a fresh checkout reports "start state in
+         collision" with no obvious cause. At z = -0.17 the 0.25 m cube's top sits
+         at -0.045, leaving 4.5 cm against a default link_padding of 0.01. -->
     <xacro:cube link_name="table" connected_to="world" length="2.00" width="2.00" height="0.25" alpha="0.3">
-      <origin xyz="0 0 -0.145" rpy="0 0 0"/>
+      <origin xyz="0 0 -0.17" rpy="0 0 0"/>
     </xacro:cube>
     <!-- Convenience alias for motion-planning-relevant tool point. The

Commit message: gripper works in mock

File: src/kinova_gen3_mock/description/kortex_robot.xacro (robot description, xacro)
@@ -15,4 +15,9 @@
     session_inactivity_timeout_ms
     connection_inactivity_timeout_ms
+    gripper:=robotiq_2f_85
+    gripper_joint_name:=robotiq_85_left_knuckle_joint
+    gripper_max_velocity:=100.0
+    gripper_max_force:=100.0
+    use_internal_bus_gripper_comm:=false
     use_fake_hardware:=false
     fake_sensor_commands:=false
@@ -44,20 +49,38 @@
       sim_gazebo="${sim_gazebo}"
       sim_isaac="${sim_isaac}"
-      gripper=""
-      gripper_joint_name=""
+      gripper="${gripper}"
+      gripper_joint_name="${gripper_joint_name}"
+      gripper_max_velocity="${gripper_max_velocity}"
+      gripper_max_force="${gripper_max_force}"
+      use_internal_bus_gripper_comm="${use_internal_bus_gripper_comm}"
       use_external_cable="${use_external_cable}"
       initial_positions="${initial_positions}">
       <xacro:insert_block name="origin" />
     </xacro:load_arm>
-    <!-- Boilerplate has no gripper; expose tool_frame at the wrist. Branches
-         that add a gripper override gripper / gripper_joint_name and bring in
-         their own gripper xacro to override this section. -->
-    <link name="${prefix}tool_frame"/>
-    <joint name="${prefix}tool_frame_joint" type="fixed">
-      <origin xyz="0 0 0" rpy="0 0 0" />
-      <parent link="${prefix}${last_arm_link}" />
-      <child link="${prefix}tool_frame" />
-      <axis xyz="0 0 0" />
-    </joint>
+    <!-- If no gripper, define tool frame here -->
+    <xacro:if value="${not gripper}">
+      <link name="${prefix}tool_frame"/>
+      <joint name="${prefix}tool_frame_joint" type="fixed">
+        <origin xyz="0 0 0" rpy="0 0 0" />
+        <parent link="${prefix}${last_arm_link}" />
+        <child link="${prefix}tool_frame" />
+        <axis xyz="0 0 0" />
+      </joint>
+    </xacro:if>
+    <!-- Include and load the gripper if defined -->
+    <xacro:unless value="${not gripper}">
+      <xacro:include filename="$(find kinova_gen3_mock)/description/grippers/${gripper}/urdf/${gripper}_macro.xacro" />
+      <xacro:load_gripper
+        parent="${prefix}${last_arm_link}"
+        prefix="${prefix}"
+        use_fake_hardware="${use_fake_hardware}"
+        fake_sensor_commands="${fake_sensor_commands}"
+        sim_gazebo="${sim_gazebo}"
+        sim_isaac="${sim_isaac}"
+        isaac_joint_commands="${isaac_joint_commands}"
+        isaac_joint_states="${isaac_joint_states}"
+        use_internal_bus_gripper_comm="${use_internal_bus_gripper_comm}"
+        moveit_active="${moveit_active}"/>
+    </xacro:unless>
   </xacro:macro>
 </robot>

File: src/kinova_gen3_mock/description/picknik_kinova_gen3.xacro (robot description, xacro)
@@ -5,4 +5,9 @@
     <xacro:arg name="dof" default="7" />
     <xacro:arg name="vision" default="true" />
+    <xacro:arg name="gripper" default="robotiq_2f_85" />
+    <xacro:arg name="gripper_joint_name" default="robotiq_85_left_knuckle_joint" />
+    <xacro:arg name="gripper_max_velocity" default="100.0" />
+    <xacro:arg name="gripper_max_force" default="100.0" />
+    <xacro:arg name="use_internal_bus_gripper_comm" default="false" />
     <xacro:arg name="robot_ip" default="yyy.yyy.yyy.yyy" />
     <xacro:arg name="username" default="admin" />
@@ -36,6 +41,5 @@
     <!-- convert to property to use substitution in function -->
     <xacro:property name="initial_positions_file" default="$(arg initial_positions_file)"/>
-    <!-- Load the robot. No gripper is mounted in this boilerplate config; the
-         Kinova-integrated wrist Vision Module is enabled via vision="true". -->
+    <!-- Load the robot -->
     <xacro:load_robot
       parent="world"
@@ -44,4 +48,9 @@
       dof="$(arg dof)"
       vision="$(arg vision)"
+      gripper="$(arg gripper)"
+      gripper_joint_name="$(arg gripper_joint_name)"
+      gripper_max_velocity="$(arg gripper_max_velocity)"
+      gripper_max_force="$(arg gripper_max_force)"
+      use_internal_bus_gripper_comm="$(arg use_internal_bus_gripper_comm)"
       robot_ip="$(arg robot_ip)"
       username="$(arg username)"
@@ -64,13 +73,21 @@
       <origin xyz="0 0 -0.145" rpy="0 0 0"/>
     </xacro:cube>
-    <!-- Convenience alias for motion-planning-relevant tool point. The
-         kortex_robot macro defines $(prefix)tool_frame at the wrist when no
-         gripper is mounted; we expose it as grasp_link so existing config files
-         (control, jtac, etc.) keep working when a gripper is added later. -->
-    <link name="$(arg prefix)grasp_link"/>
-    <joint name="$(arg prefix)grasp_link_joint" type="fixed">
-      <parent link="$(arg prefix)tool_frame"/>
-      <child link="$(arg prefix)grasp_link"/>
-      <origin xyz="0 0 0" rpy="0 0 0"/>
-    </joint>
+    <!-- Motion planning grasp link -->
+    <xacro:if value="${not '$(arg gripper)'}">
+      <link name="$(arg prefix)grasp_link"/>
+      <joint name="$(arg prefix)grasp_link_joint" type="fixed">
+        <parent link="$(arg prefix)tool_frame"/>
+        <child link="$(arg prefix)grasp_link"/>
+        <origin xyz="0 0 0" rpy="0 0 0"/>
+      </joint>
+    </xacro:if>
+    <xacro:unless value="${not '$(arg gripper)'}">
+      <!-- When gripper is mounted, attach grasp_link at the TCP of the gripper -->
+      <link name="$(arg prefix)grasp_link"/>
+      <joint name="$(arg prefix)grasp_link_joint" type="fixed">
+        <parent link="$(arg prefix)robotiq_85_base_link"/>
+        <child link="$(arg prefix)grasp_link"/>
+        <origin xyz="0 0 0.134" rpy="0 0 0"/>
+      </joint>
+    </xacro:unless>
 </robot>
