Commit message: feat(kinova_gen3): add the Robotiq 2F-85 as an opt-in gripper
The Robotiq 2F-85 is a Kinova Gen3 configuration option, so the boilerplate
offers it behind one urdf_param instead of pointing users at the
picknik_006_gen3 branch to assemble it themselves.

- gripper urdf_param (none | robotiq_2f_85) replaces gripper,
  gripper_joint_name and use_internal_bus_gripper_comm; the joint name and
  internal-bus wiring follow from it. With robotiq_2f_85 the URDF mounts
  robotiq_description's 2F-85 on end_effector_link and moves grasp_link
  0.15 m out from the gripper base. robotiq_description's macro is called
  directly: kortex_description's load_gripper wrapper passes a sim_ignition
  argument the pinned robotiq_description rejects.
- Gripper hardware follows hardware_interface: robotiq_description's mock
  block for mock, the Kortex driver over the internal bus for physical, and
  a gripper MuJoCo scene (mujoco_model_robotiq_2f_85) for mujoco.
- The SRDF becomes picknik_kinova_gen3.srdf.xacro, which MoveIt Pro runs
  through xacro with the urdf_params: a gripper group, open/close states,
  the end effector, passive mimic joints, and collision exclusions for the
  gripper against itself and the bracelet.
- robotiq_gripper_controller (GripperActionController) is declared in the
  shared manifest; configs list it in their startup lists when opting in.
- Submodules: PickNikRobotics/ros2_robotiq_gripper (main, a74d007) and
  tylerjw/serial (ros2, d8d1606), which robotiq_driver needs and has no
  Jazzy rosdep rule.
- kinova_gen3_sim: gen3_7dof_robotiq_2f_85.xml is gen3_7dof.xml plus the
  2F-85 from MuJoCo Menagerie's robotiq_2f85, with its meshes (byte-
  identical, BSD-2-Clause LICENSE and NOTICE entry). Its body frames and
  right-side joint directions are re-expressed to match robotiq_description
  without moving the simulated geometry, so the joint values MuJoCo
  publishes put the URDF links on the simulated ones. The table and floor
  move to environment.xml, shared by scene.xml and scene_robotiq_2f_85.xml.
- test_mujoco_models.py: the two arm models must match outside the
  gripper, both scenes hold their keyframe, and the simulated gripper must
  match the URDF to 1 mm when open, half closed, and closed.
- MujocoSystem's frame check samples the 2F-85's mimic joints
  independently of the closed four-bar, so its joints are listed in
  ignore_joint_validation when the gripper is mounted.

With gripper none, the generated URDFs are identical to the parent
commit's apart from two comments, and the SRDFs have the same elements.

Refs PickNikRobotics/moveit_pro#18874

Co-Authored-By: Claude Opus 5.5 <noreply@anthropic.com>

File: src/kinova_gen3_mock/description/kinova_gen3_mujoco.ros2_control.xacro (robot description, xacro)
@@ -11,5 +11,6 @@
     mujoco_model_package
     mujoco_keyframe:=''
-    mujoco_viewer:=false">
+    mujoco_viewer:=false
+    ignore_joint_validation:=''">
     <ros2_control name="${name}" type="system">
       <hardware>
@@ -23,4 +24,7 @@
         <!-- Rate at which <site> transforms are published -->
         <param name="tf_publish_rate">60</param>
+        <xacro:if value="${ignore_joint_validation != ''}">
+          <param name="ignore_joint_validation">${ignore_joint_validation}</param>
+        </xacro:if>
       </hardware>
     </ros2_control>

File: src/kinova_gen3_mock/description/kortex_robot.xacro (robot description, xacro)
@@ -60,7 +60,6 @@
       <xacro:insert_block name="origin" />
     </xacro:load_arm>
-    <!-- Boilerplate has no gripper; expose tool_frame at the wrist. Branches
-         that add a gripper override gripper / gripper_joint_name and bring in
-         their own gripper xacro to override this section. -->
+    <!-- tool_frame marks the wrist flange. The optional gripper is mounted by
+         picknik_kinova_gen3.xacro, which also places grasp_link. -->
     <link name="${prefix}tool_frame"/>
     <joint name="${prefix}tool_frame_joint" type="fixed">

File: src/kinova_gen3_mock/description/picknik_kinova_gen3.xacro (robot description, xacro)
@@ -23,22 +23,26 @@
     <xacro:arg name="isaac_joint_states" default="/isaac_joint_states" />
     <xacro:arg name="use_external_cable" default="false" />
-    <!-- Gripper selection, forwarded to ros2_kortex's load_arm. The boilerplate
-         mounts no gripper, so these default to empty and tool_frame stays at the
-         wrist flange.
-         WARNING: setting these alone does NOT mount a gripper. load_arm uses them
-         for the Kortex hardware block and to add the gripper joint to
-         <ros2_control>, but contributes no links and no kinematic joint, so a
-         config that sets only these produces a model whose <ros2_control> block
-         references a joint the kinematic model does not contain. A complete
-         gripper overlay also needs a gripper description include, a gripper
-         controller in the ros2_control manifest, and a gripper group in the SRDF.
-         See "Adding a Robotiq gripper" in the workspace README, and the
-         picknik_006_gen3 branch for a reference implementation. -->
-    <xacro:arg name="gripper" default="" />
-    <xacro:arg name="gripper_joint_name" default="" />
-    <xacro:arg name="use_internal_bus_gripper_comm" default="false" />
+    <!-- Gripper mounted on the wrist:
+           none           no gripper; tool_frame and grasp_link sit at the wrist flange
+           robotiq_2f_85  Robotiq 2F-85 on the Kinova internal bus, as Kinova sells it
+         The gripper joint name and internal-bus wiring follow from this choice.
+         Selecting a gripper also needs its controller activated; see "Robotiq
+         2F-85 gripper" in the workspace README. -->
+    <xacro:arg name="gripper" default="none" />
+    <xacro:property name="gripper" value="$(arg gripper)" />
+    <xacro:unless value="${gripper in ['none', 'robotiq_2f_85']}">
+      <xacro:element xacro:name="${xacro.fatal('gripper must be none or robotiq_2f_85, not ' + gripper)}"/>
+    </xacro:unless>
+    <!-- ros2_kortex's macros take an empty gripper name for "no gripper". -->
+    <xacro:property name="kortex_gripper" value="${'' if gripper == 'none' else gripper}" />
+    <xacro:property name="gripper_joint_name" value="${'robotiq_85_left_knuckle_joint' if gripper == 'robotiq_2f_85' else ''}" />
+    <xacro:property name="use_internal_bus_gripper_comm" value="${'true' if gripper == 'robotiq_2f_85' else 'false'}" />
     <!-- MuJoCo args, used only when hardware_interface is mujoco. The config that
          selects MuJoCo (kinova_gen3_sim) names its own scene package and file. -->
     <xacro:arg name="mujoco_model" default="" />
+    <!-- Scene simulated instead of mujoco_model when the Robotiq 2F-85 is
+         mounted, since the gripper adds bodies, joints and an actuator. -->
+    <xacro:arg name="mujoco_model_robotiq_2f_85" default="" />
+    <xacro:property name="mujoco_model" value="${xacro.arg('mujoco_model_robotiq_2f_85') if gripper == 'robotiq_2f_85' else xacro.arg('mujoco_model')}" />
     <xacro:arg name="mujoco_model_package" default="" />
     <xacro:arg name="mujoco_keyframe" default="" />
@@ -76,30 +80,39 @@
         session_inactivity_timeout_ms="$(arg session_inactivity_timeout_ms)"
         connection_inactivity_timeout_ms="$(arg connection_inactivity_timeout_ms)"
-        use_internal_bus_gripper_comm="$(arg use_internal_bus_gripper_comm)"
+        use_internal_bus_gripper_comm="${use_internal_bus_gripper_comm}"
         gripper_max_velocity="100.0"
         gripper_max_force="100.0"
-        gripper_joint_name="$(arg gripper_joint_name)"
-        gripper="$(arg gripper)"/>
+        gripper_joint_name="${gripper_joint_name}"
+        gripper="${kortex_gripper}"/>
     </xacro:if>
     <xacro:if value="${hardware_interface == 'mujoco'}">
+      <!-- MujocoSystem's startup check poses each URDF joint independently and
+           compares link frames without MuJoCo's equality constraints. The 2F-85's
+           four-bar linkage is closed by one, and its fingertips hang from a
+           different link in the MJCF than in the URDF, so off the constraint the
+           check reports mismatches the simulated gripper never has. Its joints
+           are left out of the check; kinova_gen3_sim's test_mujoco_models.py
+           compares the constrained gripper against the URDF instead. -->
+      <xacro:property name="mujoco_ignore_joint_validation" value="${'robotiq_85_left_knuckle_joint robotiq_85_right_knuckle_joint robotiq_85_left_inner_knuckle_joint robotiq_85_right_inner_knuckle_joint robotiq_85_left_finger_tip_joint robotiq_85_right_finger_tip_joint' if gripper == 'robotiq_2f_85' else ''}" />
       <xacro:include filename="$(find kinova_gen3_mock)/description/kinova_gen3_mujoco.ros2_control.xacro" />
       <xacro:kinova_gen3_mujoco_ros2_control
         name="$(arg prefix)KinovaGen3MujocoSystem"
-        mujoco_model="$(arg mujoco_model)"
+        mujoco_model="${mujoco_model}"
         mujoco_model_package="$(arg mujoco_model_package)"
         mujoco_keyframe="$(arg mujoco_keyframe)"
-        mujoco_viewer="$(arg mujoco_viewer)"/>
+        mujoco_viewer="$(arg mujoco_viewer)"
+        ignore_joint_validation="${mujoco_ignore_joint_validation}"/>
     </xacro:if>
     <xacro:unless value="${hardware_interface in ['mock', 'mujoco', 'physical']}">
       <xacro:element xacro:name="${xacro.fatal('hardware_interface must be mock, mujoco, or physical, not ' + hardware_interface)}"/>
     </xacro:unless>
-    <!-- Load the robot. No gripper is mounted by default; the Kinova-integrated
-         wrist Vision Module is enabled via vision="true". -->
+    <!-- Load the robot. The Kinova-integrated wrist Vision Module is enabled via
+         vision="true"; the gripper, if any, is loaded below. -->
     <xacro:load_robot
       parent="world"
       prefix="$(arg prefix)"
       arm="$(arg arm)"
-      gripper="$(arg gripper)"
-      gripper_joint_name="$(arg gripper_joint_name)"
+      gripper="${kortex_gripper}"
+      gripper_joint_name="${gripper_joint_name}"
       dof="$(arg dof)"
       vision="$(arg vision)"
@@ -111,5 +124,5 @@
       session_inactivity_timeout_ms="$(arg session_inactivity_timeout_ms)"
       connection_inactivity_timeout_ms="$(arg connection_inactivity_timeout_ms)"
-      use_internal_bus_gripper_comm="$(arg use_internal_bus_gripper_comm)"
+      use_internal_bus_gripper_comm="${use_internal_bus_gripper_comm}"
       use_external_cable="$(arg use_external_cable)"
       initial_positions="${xacro.load_yaml(initial_positions_file)}"
@@ -125,13 +138,39 @@
       <origin xyz="0 0 -0.17" rpy="0 0 0"/>
     </xacro:cube>
-    <!-- Convenience alias for motion-planning-relevant tool point. The
-         kortex_robot macro defines $(prefix)tool_frame at the wrist when no
-         gripper is mounted; we expose it as grasp_link so existing config files
-         (control, jtac, etc.) keep working when a gripper is added later. -->
+    <!-- Robotiq 2F-85 on the wrist flange. robotiq_description's own macro is
+         used rather than kortex_description's load_gripper wrapper, which passes a
+         sim_ignition argument the pinned robotiq_description no longer accepts.
+         Only mock hardware gets the gripper's own <ros2_control> block (mock
+         components). On the real arm the gripper joint is part of the Kortex
+         hardware block above (internal bus), and MuJoCo simulates it from the
+         gripper scene the MuJoCo block loads. -->
+    <xacro:if value="${gripper == 'robotiq_2f_85'}">
+      <xacro:include filename="$(find robotiq_description)/urdf/robotiq_2f_85_macro.urdf.xacro" />
+      <xacro:robotiq_gripper
+        name="RobotiqGripperHardwareInterface"
+        prefix="$(arg prefix)"
+        parent="$(arg prefix)end_effector_link"
+        include_ros2_control="${hardware_interface == 'mock'}"
+        use_fake_hardware="${hardware_interface == 'mock'}"
+        mock_sensor_commands="$(arg fake_sensor_commands)">
+        <origin xyz="0 0 0" rpy="0 0 0" />
+      </xacro:robotiq_gripper>
+    </xacro:if>
+    <!-- grasp_link is the motion-planning tool point that the control, JTAC and
+         SRDF configuration name. With no gripper it is tool_frame at the wrist
+         flange; with the 2F-85 it is between the fingertips, 0.15 m out from the
+         gripper base. -->
     <link name="$(arg prefix)grasp_link"/>
     <joint name="$(arg prefix)grasp_link_joint" type="fixed">
-      <parent link="$(arg prefix)tool_frame"/>
-      <child link="$(arg prefix)grasp_link"/>
-      <origin xyz="0 0 0" rpy="0 0 0"/>
+      <xacro:if value="${gripper == 'none'}">
+        <parent link="$(arg prefix)tool_frame"/>
+        <child link="$(arg prefix)grasp_link"/>
+        <origin xyz="0 0 0" rpy="0 0 0"/>
+      </xacro:if>
+      <xacro:if value="${gripper == 'robotiq_2f_85'}">
+        <parent link="$(arg prefix)robotiq_85_base_link"/>
+        <child link="$(arg prefix)grasp_link"/>
+        <origin xyz="0 0 0.15" rpy="0 0 0"/>
+      </xacro:if>
     </joint>
 </robot>
