Commit message: refactor(kinova_gen3): drop the table and the picknik_accessories submodule
A hardware vendor's boilerplate models the vendor's arm, not a work cell,
so the URDF no longer adds a 2 x 2 m table from picknik_accessories' cube
macro. The MuJoCo scene drops its matching table and puts the floor at the
arm's mounting surface (z = 0), so the simulation still matches the URDF.

That cube was the only live use of picknik_accessories, which is moving
away from holding robot assets. simulation_scene.urdf.xacro, which included
two of its furniture models, was never included by anything and is deleted.
With picknik_accessories gone, the fanuc submodule that existed only to
satisfy its rosdep on fanuc_lrmate200id_support goes too.

The generated URDFs lose only the table link and joint.

Refs PickNikRobotics/moveit_pro#18874

Co-Authored-By: Claude Opus 5.5 <noreply@anthropic.com>

File: src/kinova_gen3_mock/description/picknik_kinova_gen3.xacro (robot description, xacro)
@@ -46,7 +46,5 @@
     <!-- Import macros for main hardware components -->
     <xacro:include filename="$(find kinova_gen3_mock)/description/kortex_robot.xacro" />
-    <!-- Import environment macros -->
-    <xacro:include filename="$(find picknik_accessories)/descriptions/geometry/cube.urdf.xacro"/>
-    <!-- World is centered under base_link of the robot, on the ground -->
+    <!-- World is centered under base_link of the robot, on its mounting surface -->
     <link name="world"/>
     <!-- initial position for simulations (Mock Hardware, Gazebo, Ignition) -->
@@ -117,12 +115,4 @@
       <origin xyz="0 0 0.0" rpy="0 0 0" />
     </xacro:load_robot>
-    <!-- Environment -->
-    <!-- The table top must stay clear of base_link by more than the collision
-         padding applied to both, or a fresh checkout reports "start state in
-         collision" with no obvious cause. At z = -0.17 the 0.25 m cube's top sits
-         at -0.045, leaving 4.5 cm against a default link_padding of 0.01. -->
-    <xacro:cube link_name="table" connected_to="world" length="2.00" width="2.00" height="0.25" alpha="0.3">
-      <origin xyz="0 0 -0.17" rpy="0 0 0"/>
-    </xacro:cube>
     <!-- Convenience alias for motion-planning-relevant tool point. The
          kortex_robot macro defines $(prefix)tool_frame at the wrist when no
