Commit message: removed support for gen3 6dof and gen3_lite, retained gen3 7dof, reduced code and simplified file structure.

File: src/kinova_gen3_mock/description/arms/gen3/7dof/urdf/gen3_macro.xacro (robot description, xacro)
@@ -5,53 +5,16 @@
   <xacro:macro name="load_arm" params="
     parent
-    dof
-    vision
     prefix
     *origin
-    robot_ip
-    username:=admin
-    password:=admin
-    port:=10000
-    port_realtime:=10001
-    session_inactivity_timeout_ms:=6000
-    connection_inactivity_timeout_ms:=2000
-    use_internal_bus_gripper_comm:=true
-    gripper
-    gripper_joint_name
-    gripper_max_velocity:=100.0
-    gripper_max_force:=100.0
-    use_fake_hardware:=false
+    dof:=7
+    vision:=true
     fake_sensor_commands:=false
-    sim_gazebo:=false
-    sim_isaac:=false
-    isaac_joint_commands:=/isaac_joint_commands
-    isaac_joint_states:=/isaac_joint_states
-    use_external_cable:=false
-    initial_positions:=${dict(joint_1=0.0,joint_2=0.0,joint_3=0.0,joint_4=0.0,joint_5=0.0,joint_6=0.0,joint_7=0.0)}
-    moveit_active:=false">
+    initial_positions:=${dict(joint_1=0.0,joint_2=0.0,joint_3=0.0,joint_4=0.0,joint_5=0.0,joint_6=0.0,joint_7=0.0)}">
     <!-- ros2 control include -->
-    <xacro:include filename="$(find kinova_gen3_mock)/description/arms/gen3/${dof}dof/urdf/kortex.ros2_control.xacro" />
+    <xacro:include filename="$(find kinova_gen3_mock)/description/arms/gen3/7dof/urdf/kortex.ros2_control.xacro" />
     <xacro:kortex_ros2_control
       name="${prefix}KortexMultiInterfaceHardware" prefix="${prefix}"
-      use_fake_hardware="${use_fake_hardware}"
       fake_sensor_commands="${fake_sensor_commands}"
-      sim_gazebo="${sim_gazebo}"
-      sim_isaac="${sim_isaac}"
-      isaac_joint_commands="${isaac_joint_commands}"
-      isaac_joint_states="${isaac_joint_states}"
-      tf_prefix=""
-      initial_positions="${initial_positions}"
-      robot_ip="${robot_ip}"
-      username="${username}"
-      password="${password}"
-      port="${port}"
-      port_realtime="${port_realtime}"
-      session_inactivity_timeout_ms="${session_inactivity_timeout_ms}"
-      connection_inactivity_timeout_ms="${connection_inactivity_timeout_ms}"
-      use_internal_bus_gripper_comm="${use_internal_bus_gripper_comm}"
-      gripper_max_velocity="${gripper_max_velocity}"
-      gripper_max_force="${gripper_max_force}"
-      gripper_joint_name="${gripper_joint_name}"
-      gripper="${gripper}"/>
+      initial_positions="${initial_positions}"/>
     <joint name="${prefix}base_joint" type="fixed">
       <xacro:insert_block name="origin" />
@@ -103,38 +66,18 @@
       </collision>
     </link>
-    <xacro:if value="${use_external_cable}">
-      <joint
+    <joint
       name="${prefix}joint_1"
-      type="revolute">
-        <origin xyz="0 0 0.15643" rpy="3.1416 2.7629E-18 -4.9305E-36" />
-        <parent
-          link="${prefix}base_link" />
-        <child
-          link="${prefix}shoulder_link" />
-        <axis
-          xyz="0 0 1" />
-        <limit
-          lower="${-2*pi}"
-          upper="${2*pi}"
-          effort="39"
-          velocity="1.3963" />
-      </joint>
-    </xacro:if>
-    <xacro:unless value="${use_external_cable}">
-      <joint
-        name="${prefix}joint_1"
-        type="continuous">
-        <origin xyz="0 0 0.15643" rpy="3.1416 2.7629E-18 -4.9305E-36" />
-        <parent
-          link="${prefix}base_link" />
-        <child
-          link="${prefix}shoulder_link" />
-        <axis
-          xyz="0 0 1" />
-        <limit
-          effort="39"
-          velocity="1.3963" />
-      </joint>
-    </xacro:unless>
+      type="continuous">
+      <origin xyz="0 0 0.15643" rpy="3.1416 2.7629E-18 -4.9305E-36" />
+      <parent
+        link="${prefix}base_link" />
+      <child
+        link="${prefix}shoulder_link" />
+      <axis
+        xyz="0 0 1" />
+      <limit
+        effort="39"
+        velocity="1.3963" />
+    </joint>
     <link name="${prefix}half_arm_1_link">
       <inertial>
@@ -193,38 +136,18 @@
       </collision>
     </link>
-    <xacro:if value="${use_external_cable}">
-      <joint
-        name="${prefix}joint_3"
-        type="revolute">
-        <origin xyz="0 -0.21038 -0.006375" rpy="-1.5708 1.2326E-32 -2.9122E-16" />
-        <parent
-          link="${prefix}half_arm_1_link" />
-        <child
-          link="${prefix}half_arm_2_link" />
-        <axis
-          xyz="0 0 1" />
-        <limit
-          lower="${-2*pi}"
-          upper="${2*pi}"
-          effort="39"
-          velocity="1.3963" />
-      </joint>
-    </xacro:if>
-    <xacro:unless value="${use_external_cable}">
-      <joint
-        name="${prefix}joint_3"
-        type="continuous">
-        <origin xyz="0 -0.21038 -0.006375" rpy="-1.5708 1.2326E-32 -2.9122E-16" />
-        <parent
-          link="${prefix}half_arm_1_link" />
-        <child
-          link="${prefix}half_arm_2_link" />
-        <axis
-          xyz="0 0 1" />
-        <limit
-          effort="39"
-          velocity="1.3963" />
-      </joint>
-    </xacro:unless>
+    <joint
+      name="${prefix}joint_3"
+      type="continuous">
+      <origin xyz="0 -0.21038 -0.006375" rpy="-1.5708 1.2326E-32 -2.9122E-16" />
+      <parent
+        link="${prefix}half_arm_1_link" />
+      <child
+        link="${prefix}half_arm_2_link" />
+      <axis
+        xyz="0 0 1" />
+      <limit
+        effort="39"
+        velocity="1.3963" />
+    </joint>
     <link name="${prefix}forearm_link">
       <inertial>
@@ -283,38 +206,18 @@
       </collision>
     </link>
-    <xacro:if value="${use_external_cable}">
-      <joint
-        name="${prefix}joint_5"
-        type="revolute">
-        <origin xyz="0 -0.20843 -0.006375" rpy="-1.5708 2.2204E-16 -6.373E-17" />
-        <parent
-          link="${prefix}forearm_link" />
-        <child
-          link="${prefix}spherical_wrist_1_link" />
-        <axis
-          xyz="0 0 1" />
-        <limit
-          lower="${-2*pi}"
-          upper="${2*pi}"
-          effort="9"
-          velocity="1.2218" />
-      </joint>
-    </xacro:if>
-    <xacro:unless value="${use_external_cable}">
-      <joint
-        name="${prefix}joint_5"
-        type="continuous">
-        <origin xyz="0 -0.20843 -0.006375" rpy="-1.5708 2.2204E-16 -6.373E-17" />
-        <parent
-          link="${prefix}forearm_link" />
-        <child
-          link="${prefix}spherical_wrist_1_link" />
-        <axis
-          xyz="0 0 1" />
-        <limit
-          effort="9"
-          velocity="1.2218" />
-      </joint>
-    </xacro:unless>
+    <joint
+      name="${prefix}joint_5"
+      type="continuous">
+      <origin xyz="0 -0.20843 -0.006375" rpy="-1.5708 2.2204E-16 -6.373E-17" />
+      <parent
+        link="${prefix}forearm_link" />
+      <child
+        link="${prefix}spherical_wrist_1_link" />
+      <axis
+        xyz="0 0 1" />
+      <limit
+        effort="9"
+        velocity="1.2218" />
+    </joint>
     <link name="${prefix}spherical_wrist_2_link">
       <inertial>
@@ -399,38 +302,18 @@
     </link>
     </xacro:unless>
-    <xacro:if value="${use_external_cable}">
-      <joint
-        name="${prefix}joint_7"
-        type="revolute">
-        <origin xyz="0 -0.10593 -0.00017505" rpy="-1.5708 -5.5511E-17 9.6396E-17" />
-        <parent
-          link="${prefix}spherical_wrist_2_link" />
-        <child
-          link="${prefix}bracelet_link" />
-        <axis
-          xyz="0 0 1" />
-        <limit
-          lower="${-2*pi}"
-          upper="${2*pi}"
-          effort="9"
-          velocity="1.2218" />
-      </joint>
-    </xacro:if>
-    <xacro:unless value="${use_external_cable}">
-      <joint
-        name="${prefix}joint_7"
-        type="continuous">
-        <origin xyz="0 -0.10593 -0.00017505" rpy="-1.5708 -5.5511E-17 9.6396E-17" />
-        <parent
-          link="${prefix}spherical_wrist_2_link" />
-        <child
-          link="${prefix}bracelet_link" />
-        <axis
-          xyz="0 0 1" />
-        <limit
-          effort="9"
-          velocity="1.2218" />
-      </joint>
-    </xacro:unless>
+    <joint
+      name="${prefix}joint_7"
+      type="continuous">
+      <origin xyz="0 -0.10593 -0.00017505" rpy="-1.5708 -5.5511E-17 9.6396E-17" />
+      <parent
+        link="${prefix}spherical_wrist_2_link" />
+      <child
+        link="${prefix}bracelet_link" />
+      <axis
+        xyz="0 0 1" />
+      <limit
+        effort="9"
+        velocity="1.2218" />
+    </joint>
     <link name="${prefix}end_effector_link" />
     <joint
@@ -446,45 +329,22 @@
     </joint>
     <xacro:if value="${vision}">
-      <!-- sim camera needs to be rotated which might not apply to built in vision module -->
-      <xacro:if value="${sim_gazebo}">
-        <link name="${prefix}camera_link" />
-        <joint name="${prefix}camera_module" type="fixed">
-          <origin xyz="0 0.05639 0.01305" rpy="0 ${-pi/2} ${-pi/2}" />
-          <parent link="${prefix}end_effector_link" />
-          <child  link="${prefix}camera_link" />
-        </joint>
-        <link name="${prefix}camera_depth_frame" />
-        <joint name="${prefix}depth_module" type="fixed">
-          <origin xyz="0.0275 0.066 0.01305" rpy="0 ${-pi/2} ${-pi/2}" />
-          <parent link="${prefix}end_effector_link" />
-          <child  link="${prefix}camera_depth_frame" />
-        </joint>
-        <link name="${prefix}camera_color_frame" />
-        <joint name="${prefix}color_module" type="fixed">
-          <origin xyz="0 0.05639 0.01305" rpy="0 ${-pi/2} ${-pi/2}" />
-          <parent link="${prefix}end_effector_link" />
-          <child  link="${prefix}camera_color_frame" />
-        </joint>
-      </xacro:if>
-      <xacro:unless value="${sim_gazebo}">
-        <link name="${prefix}camera_link" />
-        <joint name="${prefix}camera_module" type="fixed">
-          <origin xyz="0 0.05639 -0.00305" rpy="${pi} ${pi} 0" />
-          <parent link="${prefix}end_effector_link" />
-          <child  link="${prefix}camera_link" />
-        </joint>
-        <link name="${prefix}camera_depth_frame" />
-        <joint name="${prefix}depth_module" type="fixed">
-          <origin xyz="0.0275 0.066 -0.00305" rpy="${pi} ${pi} 0" />
-          <parent link="${prefix}end_effector_link" />
-          <child  link="${prefix}camera_depth_frame" />
-        </joint>
-        <link name="${prefix}camera_color_frame" />
-        <joint name="${prefix}color_module" type="fixed">
-          <origin xyz="0 0.05639 -0.00305" rpy="${pi} ${pi} 0" />
-          <parent link="${prefix}end_effector_link" />
-          <child  link="${prefix}camera_color_frame" />
-        </joint>
-      </xacro:unless>
+      <link name="${prefix}camera_link" />
+      <joint name="${prefix}camera_module" type="fixed">
+        <origin xyz="0 0.05639 -0.00305" rpy="${pi} ${pi} 0" />
+        <parent link="${prefix}end_effector_link" />
+        <child  link="${prefix}camera_link" />
+      </joint>
+      <link name="${prefix}camera_depth_frame" />
+      <joint name="${prefix}depth_module" type="fixed">
+        <origin xyz="0.0275 0.066 -0.00305" rpy="${pi} ${pi} 0" />
+        <parent link="${prefix}end_effector_link" />
+        <child  link="${prefix}camera_depth_frame" />
+      </joint>
+      <link name="${prefix}camera_color_frame" />
+      <joint name="${prefix}color_module" type="fixed">
+        <origin xyz="0 0.05639 -0.00305" rpy="${pi} ${pi} 0" />
+        <parent link="${prefix}end_effector_link" />
+        <child  link="${prefix}camera_color_frame" />
+      </joint>
     </xacro:if>
   </xacro:macro>

File: src/kinova_gen3_mock/description/arms/gen3/7dof/urdf/kortex.ros2_control.xacro (robot description, xacro)
@@ -4,55 +4,11 @@
     name
     prefix
-    use_fake_hardware:=false
     fake_sensor_commands:=false
-    sim_gazebo:=false
-    sim_isaac:=false
-    isaac_joint_commands:=/isaac_joint_commands
-    isaac_joint_states:=/isaac_joint_states
-    use_internal_bus_gripper_comm:=true
-    tf_prefix
-    initial_positions:=${dict(joint_1=0.0,joint_2=0.0,joint_3=0.0,joint_4=0.0,joint_5=0.0,joint_6=0.0,joint_7=0.0)}
-    robot_ip
-    username
-    password
-    port
-    port_realtime
-    session_inactivity_timeout_ms
-    connection_inactivity_timeout_ms
-    gripper
-    gripper_joint_name
-    gripper_max_velocity:=100.0
-    gripper_max_force:=100.0
-    moveit_active:=false">
+    initial_positions:=${dict(joint_1=0.0,joint_2=0.0,joint_3=0.0,joint_4=0.0,joint_5=0.0,joint_6=0.0,joint_7=0.0)}">
     <ros2_control name="${name}" type="system">
       <hardware>
-        <xacro:if value="${sim_gazebo}">
-          <plugin>gz_ros2_control/GazeboSimSystem</plugin>
-        </xacro:if>
-        <xacro:if value="${sim_isaac}">
-          <plugin>topic_based_ros2_control/TopicBasedSystem</plugin>
-          <param name="joint_commands_topic">${isaac_joint_commands}</param>
-          <param name="joint_states_topic">${isaac_joint_states}</param>
-        </xacro:if>
-        <xacro:if value="${use_fake_hardware}">
-          <plugin>mock_components/GenericSystem</plugin>
-          <param name="fake_sensor_commands">${fake_sensor_commands}</param>
-          <param name="state_following_offset">0.0</param>
-        </xacro:if>
-        <xacro:unless value="${use_fake_hardware or sim_gazebo or sim_isaac}">
-          <plugin>kortex_driver/KortexMultiInterfaceHardware</plugin>
-          <param name="robot_ip">${robot_ip}</param>
-          <param name="username">${username}</param>
-          <param name="password">${password}</param>
-          <param name="port">${port}</param>
-          <param name="port_realtime">${port_realtime}</param>
-          <param name="session_inactivity_timeout_ms">${session_inactivity_timeout_ms}</param>
-          <param name="connection_inactivity_timeout_ms">${connection_inactivity_timeout_ms}</param>
-          <param name="tf_prefix">"${tf_prefix}"</param>
-          <param name="use_internal_bus_gripper_comm">${use_internal_bus_gripper_comm}</param>
-          <param name="gripper_joint_name">${gripper_joint_name}</param>
-          <param name="gripper_max_velocity">${gripper_max_velocity}</param>
-          <param name="gripper_max_force">${gripper_max_force}</param>
-        </xacro:unless>
+        <plugin>mock_components/GenericSystem</plugin>
+        <param name="fake_sensor_commands">${fake_sensor_commands}</param>
+        <param name="state_following_offset">0.0</param>
       </hardware>
       <joint name="${prefix}joint_1">
@@ -133,15 +89,4 @@
         <state_interface name="effort"/>
       </joint>
-      <xacro:unless value="${use_fake_hardware or sim_gazebo or sim_isaac}">
-      <xacro:unless value="${not gripper}">
-        <xacro:if value="${use_internal_bus_gripper_comm}">
-          <joint name="${prefix}${gripper_joint_name}">
-            <command_interface name="position" />
-            <state_interface name="position"/>
-            <state_interface name="velocity"/>
-          </joint>
-        </xacro:if>
-      </xacro:unless>
-      </xacro:unless>
       <!-- These state values are set in order for the robot to be teleoperable in mock with the VFC -->
       <sensor name="fts">

File: src/kinova_gen3_mock/description/grippers/robotiq_2f_85/urdf/robotiq_2f_85_macro.xacro (robot description, xacro)
@@ -4,29 +4,14 @@
     parent
     prefix
-    use_fake_hardware:=false
-    fake_sensor_commands:=false
-    sim_gazebo:=false
-    sim_isaac:=false
-    isaac_joint_commands:=/isaac_joint_commands
-    isaac_joint_states:=/isaac_joint_states
-    use_internal_bus_gripper_comm:=false
-    com_port:=/dev/ttyUSB0
-    moveit_active:=false">
+    fake_sensor_commands:=false">
     <xacro:include filename="$(find robotiq_description)/urdf/robotiq_2f_85_macro.urdf.xacro" />
-    <!-- Hardware talks directly to the gripper so we don't need ros2_control unless we are simulating -->
-    <xacro:property name="include_ros2_control" value="false"/>
-    <xacro:if value="${sim_gazebo or sim_isaac or use_fake_hardware or not use_internal_bus_gripper_comm}">
-      <xacro:property name="include_ros2_control" value="true"/>
-    </xacro:if>
     <xacro:robotiq_gripper
         name="RobotiqGripperHardwareInterface"
         prefix="${prefix}"
         parent="${parent}"
-        include_ros2_control="${include_ros2_control}"
-        com_port="${com_port}"
-        use_fake_hardware="${use_fake_hardware}"
-        fake_sensor_commands="${fake_sensor_commands}"
-        sim_ignition="${sim_gazebo}"
-        sim_isaac="${sim_isaac}">
+        include_ros2_control="true"
+        com_port="/dev/ttyUSB0"
+        use_fake_hardware="true"
+        fake_sensor_commands="${fake_sensor_commands}">
         <origin xyz="0 0 0" rpy="0 0 0" />
     </xacro:robotiq_gripper>

File: src/kinova_gen3_mock/description/kortex_robot.xacro (robot description, xacro)
@@ -4,83 +4,25 @@
     parent
     *origin
-    prefix
-    arm
-    dof
-    vision
-    robot_ip
-    username
-    password
-    port
-    port_realtime
-    session_inactivity_timeout_ms
-    connection_inactivity_timeout_ms
-    gripper:=robotiq_2f_85
-    gripper_joint_name:=robotiq_85_left_knuckle_joint
-    gripper_max_velocity:=100.0
-    gripper_max_force:=100.0
-    use_internal_bus_gripper_comm:=false
-    use_fake_hardware:=false
+    prefix:=''
+    vision:=true
     fake_sensor_commands:=false
-    sim_gazebo:=false
-    sim_ignition:=false
-    sim_isaac:=false
-    isaac_joint_commands:=/isaac_joint_commands
-    isaac_joint_states:=/isaac_joint_states
-    use_external_cable:=false
-    initial_positions:=${dict(joint_1=0.0,joint_2=0.0,joint_3=0.0,joint_4=0.0,joint_5=0.0,joint_6=0.0,joint_7=0.0)}
-    moveit_active:=false">
+    initial_positions:=${dict(joint_1=0.0,joint_2=0.0,joint_3=0.0,joint_4=0.0,joint_5=0.0,joint_6=0.0,joint_7=0.0)}">
     <!-- Include and load arm macro files -->
-    <xacro:include filename="$(find kinova_gen3_mock)/description/arms/${arm}/${dof}dof/urdf/${arm}_macro.xacro" />
+    <xacro:include filename="$(find kinova_gen3_mock)/description/arms/gen3/7dof/urdf/gen3_macro.xacro" />
     <!-- Load the arm -->
     <xacro:load_arm
       parent="${parent}"
-      dof="${dof}"
       vision="${vision}"
-      robot_ip="${robot_ip}"
-      username="${username}"
-      password="${password}"
-      port="${port}"
-      port_realtime="${port_realtime}"
-      session_inactivity_timeout_ms="${session_inactivity_timeout_ms}"
-      connection_inactivity_timeout_ms="${connection_inactivity_timeout_ms}"
       prefix="${prefix}"
-      use_fake_hardware="${use_fake_hardware}"
       fake_sensor_commands="${fake_sensor_commands}"
-      sim_gazebo="${sim_gazebo}"
-      sim_isaac="${sim_isaac}"
-      gripper="${gripper}"
-      gripper_joint_name="${gripper_joint_name}"
-      gripper_max_velocity="${gripper_max_velocity}"
-      gripper_max_force="${gripper_max_force}"
-      use_internal_bus_gripper_comm="${use_internal_bus_gripper_comm}"
-      use_external_cable="${use_external_cable}"
       initial_positions="${initial_positions}">
       <xacro:insert_block name="origin" />
     </xacro:load_arm>
-    <!-- If no gripper, define tool frame here -->
-    <xacro:if value="${not gripper}">
-      <link name="${prefix}tool_frame"/>
-      <joint name="${prefix}tool_frame_joint" type="fixed">
-        <origin xyz="0 0 0" rpy="0 0 0" />
-        <parent link="${prefix}${last_arm_link}" />
-        <child link="${prefix}tool_frame" />
-        <axis xyz="0 0 0" />
-      </joint>
-    </xacro:if>
-    <!-- Include and load the gripper if defined -->
-    <xacro:unless value="${not gripper}">
-      <xacro:include filename="$(find kinova_gen3_mock)/description/grippers/${gripper}/urdf/${gripper}_macro.xacro" />
-      <xacro:load_gripper
-        parent="${prefix}${last_arm_link}"
-        prefix="${prefix}"
-        use_fake_hardware="${use_fake_hardware}"
-        fake_sensor_commands="${fake_sensor_commands}"
-        sim_gazebo="${sim_gazebo}"
-        sim_isaac="${sim_isaac}"
-        isaac_joint_commands="${isaac_joint_commands}"
-        isaac_joint_states="${isaac_joint_states}"
-        use_internal_bus_gripper_comm="${use_internal_bus_gripper_comm}"
-        moveit_active="${moveit_active}"/>
-    </xacro:unless>
+    <!-- Include and load the gripper -->
+    <xacro:include filename="$(find kinova_gen3_mock)/description/grippers/robotiq_2f_85/urdf/robotiq_2f_85_macro.xacro" />
+    <xacro:load_gripper
+      parent="${prefix}${last_arm_link}"
+      prefix="${prefix}"
+      fake_sensor_commands="${fake_sensor_commands}"/>
   </xacro:macro>
 </robot>
