Commit message: removed support for gen3 6dof and gen3_lite, retained gen3 7dof, reduced code and simplified file structure.

File: src/kinova_gen3_mock/description/picknik_kinova_gen3.xacro (robot description, xacro)
@@ -2,33 +2,7 @@
 <robot name="gen3" xmlns:xacro="http://ros.org/wiki/xacro">
     <!-- Arguments for Kinova -->
-    <xacro:arg name="arm" default="gen3" />
-    <xacro:arg name="dof" default="7" />
+    <xacro:arg name="prefix" default="" />
     <xacro:arg name="vision" default="true" />
-    <xacro:arg name="gripper" default="robotiq_2f_85" />
-    <xacro:arg name="gripper_joint_name" default="robotiq_85_left_knuckle_joint" />
-    <xacro:arg name="gripper_max_velocity" default="100.0" />
-    <xacro:arg name="gripper_max_force" default="100.0" />
-    <xacro:arg name="use_internal_bus_gripper_comm" default="false" />
-    <xacro:arg name="robot_ip" default="yyy.yyy.yyy.yyy" />
-    <xacro:arg name="username" default="admin" />
-    <xacro:arg name="password" default="admin" />
-    <xacro:arg name="port" default="10000" />
-    <xacro:arg name="port_realtime" default="10001" />
-    <xacro:arg name="session_inactivity_timeout_ms" default="60000" />
-    <xacro:arg name="connection_inactivity_timeout_ms" default="2000" />
-    <xacro:arg name="prefix" default="" />
-    <xacro:arg name="use_fake_hardware" default="true" />
     <xacro:arg name="fake_sensor_commands" default="false" />
-    <xacro:arg name="sim_gazebo" default="false" />
-    <xacro:arg name="sim_ignition" default="false" />
-    <xacro:arg name="sim_isaac" default="false" />
-    <xacro:arg name="isaac_joint_commands" default="/isaac_joint_commands" />
-    <xacro:arg name="isaac_joint_states" default="/isaac_joint_states" />
-    <xacro:arg name="use_external_cable" default="false" />
-    <!-- Simulator-specific args (no-ops for mock and hw; consumed by inheriting
-         configs that select a MuJoCo or Isaac scene). -->
-    <xacro:arg name="mujoco_model" default="" />
-    <xacro:arg name="mujoco_keyframe" default="" />
-    <xacro:arg name="mujoco_viewer" default="false" />
     <!-- Import macros for main hardware components -->
     <xacro:include filename="$(find kinova_gen3_mock)/description/kortex_robot.xacro" />
@@ -37,7 +11,6 @@
     <!-- World is centered under base_link of the robot, on the ground -->
     <link name="world"/>
-    <!-- initial position for simulations (Mock Hardware, Gazebo, Ignition) -->
+    <!-- Initial position for mock simulation -->
     <xacro:arg name="initial_positions_file" default="$(find kinova_gen3_mock)/config/initial_positions.yaml"/>
-    <!-- convert to property to use substitution in function -->
     <xacro:property name="initial_positions_file" default="$(arg initial_positions_file)"/>
     <!-- Load the robot -->
@@ -45,25 +18,6 @@
       parent="world"
       prefix="$(arg prefix)"
-      arm="$(arg arm)"
-      dof="$(arg dof)"
       vision="$(arg vision)"
-      gripper="$(arg gripper)"
-      gripper_joint_name="$(arg gripper_joint_name)"
-      gripper_max_velocity="$(arg gripper_max_velocity)"
-      gripper_max_force="$(arg gripper_max_force)"
-      use_internal_bus_gripper_comm="$(arg use_internal_bus_gripper_comm)"
-      robot_ip="$(arg robot_ip)"
-      username="$(arg username)"
-      password="$(arg password)"
-      port="$(arg port)"
-      port_realtime="$(arg port_realtime)"
-      session_inactivity_timeout_ms="$(arg session_inactivity_timeout_ms)"
-      connection_inactivity_timeout_ms="$(arg connection_inactivity_timeout_ms)"
-      use_fake_hardware="$(arg use_fake_hardware)"
       fake_sensor_commands="$(arg fake_sensor_commands)"
-      sim_gazebo="$(arg sim_gazebo)"
-      sim_ignition="$(arg sim_ignition)"
-      sim_isaac="$(arg sim_isaac)"
-      use_external_cable="$(arg use_external_cable)"
       initial_positions="${xacro.load_yaml(initial_positions_file)}" >
       <origin xyz="0 0 0.0" rpy="0 0 0" />
@@ -73,21 +27,10 @@
       <origin xyz="0 0 -0.145" rpy="0 0 0"/>
     </xacro:cube>
-    <!-- Motion planning grasp link -->
-    <xacro:if value="${not '$(arg gripper)'}">
-      <link name="$(arg prefix)grasp_link"/>
-      <joint name="$(arg prefix)grasp_link_joint" type="fixed">
-        <parent link="$(arg prefix)tool_frame"/>
-        <child link="$(arg prefix)grasp_link"/>
-        <origin xyz="0 0 0" rpy="0 0 0"/>
-      </joint>
-    </xacro:if>
-    <xacro:unless value="${not '$(arg gripper)'}">
-      <!-- When gripper is mounted, attach grasp_link at the TCP of the gripper -->
-      <link name="$(arg prefix)grasp_link"/>
-      <joint name="$(arg prefix)grasp_link_joint" type="fixed">
-        <parent link="$(arg prefix)robotiq_85_base_link"/>
-        <child link="$(arg prefix)grasp_link"/>
-        <origin xyz="0 0 0.134" rpy="0 0 0"/>
-      </joint>
-    </xacro:unless>
+    <!-- Motion planning grasp link at the TCP of the gripper -->
+    <link name="$(arg prefix)grasp_link"/>
+    <joint name="$(arg prefix)grasp_link_joint" type="fixed">
+      <parent link="$(arg prefix)robotiq_85_base_link"/>
+      <child link="$(arg prefix)grasp_link"/>
+      <origin xyz="0 0 0.134" rpy="0 0 0"/>
+    </joint>
 </robot>

Commit message: Kortex hardware interface configured

File: src/kinova_gen3_mock/description/arms/gen3/7dof/urdf/gen3_macro.xacro (robot description, xacro)
@@ -15,5 +15,18 @@
     mujoco_viewer:=false
     mujoco_keyframe:=default
-    initial_positions:=${dict(joint_1=0.0,joint_2=0.0,joint_3=0.0,joint_4=0.0,joint_5=0.0,joint_6=0.0,joint_7=0.0)}">
+    initial_positions:=${dict(joint_1=0.0,joint_2=0.0,joint_3=0.0,joint_4=0.0,joint_5=0.0,joint_6=0.0,joint_7=0.0)}
+    robot_ip:=192.168.1.10
+    username:=admin
+    password:=admin
+    port:=10000
+    port_realtime:=10001
+    session_inactivity_timeout_ms:=60000
+    connection_inactivity_timeout_ms:=2000
+    tf_prefix:=''
+    use_internal_bus_gripper_comm:=false
+    gripper:=robotiq_2f_85
+    gripper_joint_name:=robotiq_85_left_knuckle_joint
+    gripper_max_velocity:=100.0
+    gripper_max_force:=100.0">
     <!-- ros2 control include -->
     <xacro:include filename="$(find kinova_gen3_mock)/description/arms/gen3/7dof/urdf/kortex.ros2_control.xacro" />
@@ -26,5 +39,18 @@
       mujoco_viewer="${mujoco_viewer}"
       mujoco_keyframe="${mujoco_keyframe}"
-      initial_positions="${initial_positions}"/>
+      initial_positions="${initial_positions}"
+      robot_ip="${robot_ip}"
+      username="${username}"
+      password="${password}"
+      port="${port}"
+      port_realtime="${port_realtime}"
+      session_inactivity_timeout_ms="${session_inactivity_timeout_ms}"
+      connection_inactivity_timeout_ms="${connection_inactivity_timeout_ms}"
+      tf_prefix="${tf_prefix}"
+      use_internal_bus_gripper_comm="${use_internal_bus_gripper_comm}"
+      gripper="${gripper}"
+      gripper_joint_name="${gripper_joint_name}"
+      gripper_max_velocity="${gripper_max_velocity}"
+      gripper_max_force="${gripper_max_force}"/>
     <joint name="${prefix}base_joint" type="fixed">
       <xacro:insert_block name="origin" />

File: src/kinova_gen3_mock/description/arms/gen3/7dof/urdf/kortex.ros2_control.xacro (robot description, xacro)
@@ -10,24 +10,52 @@
     mujoco_viewer:=false
     mujoco_keyframe:=default
-    initial_positions:=${dict(joint_1=0.0,joint_2=0.0,joint_3=0.0,joint_4=0.0,joint_5=0.0,joint_6=0.0,joint_7=0.0)}">
+    initial_positions:=${dict(joint_1=0.0,joint_2=0.0,joint_3=0.0,joint_4=0.0,joint_5=0.0,joint_6=0.0,joint_7=0.0)}
+    robot_ip:=192.168.1.10
+    username:=admin
+    password:=admin
+    port:=10000
+    port_realtime:=10001
+    session_inactivity_timeout_ms:=60000
+    connection_inactivity_timeout_ms:=2000
+    tf_prefix:=''
+    use_internal_bus_gripper_comm:=false
+    gripper:=robotiq_2f_85
+    gripper_joint_name:=robotiq_85_left_knuckle_joint
+    gripper_max_velocity:=100.0
+    gripper_max_force:=100.0">
     <ros2_control name="${name}" type="system">
-      <xacro:if value="${use_fake_hardware}">
-        <hardware>
+      <hardware>
+        <xacro:if value="${use_fake_hardware}">
           <plugin>mock_components/GenericSystem</plugin>
           <param name="fake_sensor_commands">${fake_sensor_commands}</param>
           <param name="state_following_offset">0.0</param>
-        </hardware>
-      </xacro:if>
-      <xacro:unless value="${use_fake_hardware}">
-        <hardware>
-          <plugin>picknik_mujoco_ros/MujocoSystem</plugin>
-          <param name="mujoco_model">${mujoco_model}</param>
-          <param name="mujoco_model_package">${mujoco_model_package}</param>
-          <param name="mujoco_viewer">${mujoco_viewer}</param>
-          <param name="mujoco_keyframe">${mujoco_keyframe}</param>
-          <param name="render_publish_rate">10</param>
-          <param name="tf_publish_rate">60</param>
-        </hardware>
-      </xacro:unless>
+        </xacro:if>
+        <xacro:unless value="${use_fake_hardware}">
+          <xacro:if value="${robot_ip != '' and robot_ip != '0.0.0.0'}">
+            <plugin>kortex_driver/KortexMultiInterfaceHardware</plugin>
+            <param name="robot_ip">${robot_ip}</param>
+            <param name="username">${username}</param>
+            <param name="password">${password}</param>
+            <param name="port">${port}</param>
+            <param name="port_realtime">${port_realtime}</param>
+            <param name="session_inactivity_timeout_ms">${session_inactivity_timeout_ms}</param>
+            <param name="connection_inactivity_timeout_ms">${connection_inactivity_timeout_ms}</param>
+            <param name="tf_prefix">"${tf_prefix}"</param>
+            <param name="use_internal_bus_gripper_comm">${use_internal_bus_gripper_comm}</param>
+            <param name="gripper_joint_name">${gripper_joint_name}</param>
+            <param name="gripper_max_velocity">${gripper_max_velocity}</param>
+            <param name="gripper_max_force">${gripper_max_force}</param>
+          </xacro:if>
+          <xacro:unless value="${robot_ip != '' and robot_ip != '0.0.0.0'}">
+            <plugin>picknik_mujoco_ros/MujocoSystem</plugin>
+            <param name="mujoco_model">${mujoco_model}</param>
+            <param name="mujoco_model_package">${mujoco_model_package}</param>
+            <param name="mujoco_viewer">${mujoco_viewer}</param>
+            <param name="mujoco_keyframe">${mujoco_keyframe}</param>
+            <param name="render_publish_rate">10</param>
+            <param name="tf_publish_rate">60</param>
+          </xacro:unless>
+        </xacro:unless>
+      </hardware>
       <joint name="${prefix}joint_1">
         <command_interface name="position">
@@ -107,4 +135,17 @@
         <state_interface name="effort"/>
       </joint>
+      <xacro:unless value="${use_fake_hardware}">
+        <xacro:if value="${robot_ip != '' and robot_ip != '0.0.0.0'}">
+          <xacro:unless value="${not gripper}">
+            <xacro:if value="${use_internal_bus_gripper_comm}">
+              <joint name="${prefix}${gripper_joint_name}">
+                <command_interface name="position" />
+                <state_interface name="position"/>
+                <state_interface name="velocity"/>
+              </joint>
+            </xacro:if>
+          </xacro:unless>
+        </xacro:if>
+      </xacro:unless>
       <!-- These state values are set in order for the robot to be teleoperable in mock with the VFC -->
       <sensor name="fts">

File: src/kinova_gen3_mock/description/kortex_robot.xacro (robot description, xacro)
@@ -12,5 +12,18 @@
     mujoco_viewer:=false
     mujoco_keyframe:=default
-    initial_positions:=${dict(joint_1=0.0,joint_2=0.0,joint_3=0.0,joint_4=0.0,joint_5=0.0,joint_6=0.0,joint_7=0.0)}">
+    initial_positions:=${dict(joint_1=0.0,joint_2=0.0,joint_3=0.0,joint_4=0.0,joint_5=0.0,joint_6=0.0,joint_7=0.0)}
+    robot_ip:=192.168.1.10
+    username:=admin
+    password:=admin
+    port:=10000
+    port_realtime:=10001
+    session_inactivity_timeout_ms:=60000
+    connection_inactivity_timeout_ms:=2000
+    tf_prefix:=''
+    use_internal_bus_gripper_comm:=false
+    gripper:=robotiq_2f_85
+    gripper_joint_name:=robotiq_85_left_knuckle_joint
+    gripper_max_velocity:=100.0
+    gripper_max_force:=100.0">
     <!-- Include and load arm macro files -->
     <xacro:include filename="$(find kinova_gen3_mock)/description/arms/gen3/7dof/urdf/gen3_macro.xacro" />
@@ -26,5 +39,18 @@
       mujoco_viewer="${mujoco_viewer}"
       mujoco_keyframe="${mujoco_keyframe}"
-      initial_positions="${initial_positions}">
+      initial_positions="${initial_positions}"
+      robot_ip="${robot_ip}"
+      username="${username}"
+      password="${password}"
+      port="${port}"
+      port_realtime="${port_realtime}"
+      session_inactivity_timeout_ms="${session_inactivity_timeout_ms}"
+      connection_inactivity_timeout_ms="${connection_inactivity_timeout_ms}"
+      tf_prefix="${tf_prefix}"
+      use_internal_bus_gripper_comm="${use_internal_bus_gripper_comm}"
+      gripper="${gripper}"
+      gripper_joint_name="${gripper_joint_name}"
+      gripper_max_velocity="${gripper_max_velocity}"
+      gripper_max_force="${gripper_max_force}">
       <xacro:insert_block name="origin" />
     </xacro:load_arm>

File: src/kinova_gen3_mock/description/picknik_kinova_gen3.xacro (robot description, xacro)
@@ -10,4 +10,17 @@
     <xacro:arg name="mujoco_viewer" default="false" />
     <xacro:arg name="mujoco_keyframe" default="default" />
+    <xacro:arg name="robot_ip" default="192.168.1.10" />
+    <xacro:arg name="username" default="admin" />
+    <xacro:arg name="password" default="admin" />
+    <xacro:arg name="port" default="10000" />
+    <xacro:arg name="port_realtime" default="10001" />
+    <xacro:arg name="session_inactivity_timeout_ms" default="60000" />
+    <xacro:arg name="connection_inactivity_timeout_ms" default="2000" />
+    <xacro:arg name="tf_prefix" default="" />
+    <xacro:arg name="use_internal_bus_gripper_comm" default="false" />
+    <xacro:arg name="gripper" default="robotiq_2f_85" />
+    <xacro:arg name="gripper_joint_name" default="robotiq_85_left_knuckle_joint" />
+    <xacro:arg name="gripper_max_velocity" default="100.0" />
+    <xacro:arg name="gripper_max_force" default="100.0" />
     <!-- Import macros for main hardware components -->
     <xacro:include filename="$(find kinova_gen3_mock)/description/kortex_robot.xacro" />
@@ -30,5 +43,18 @@
       mujoco_viewer="$(arg mujoco_viewer)"
       mujoco_keyframe="$(arg mujoco_keyframe)"
-      initial_positions="${xacro.load_yaml(initial_positions_file)}" >
+      initial_positions="${xacro.load_yaml(initial_positions_file)}"
+      robot_ip="$(arg robot_ip)"
+      username="$(arg username)"
+      password="$(arg password)"
+      port="$(arg port)"
+      port_realtime="$(arg port_realtime)"
+      session_inactivity_timeout_ms="$(arg session_inactivity_timeout_ms)"
+      connection_inactivity_timeout_ms="$(arg connection_inactivity_timeout_ms)"
+      tf_prefix="$(arg tf_prefix)"
+      use_internal_bus_gripper_comm="$(arg use_internal_bus_gripper_comm)"
+      gripper="$(arg gripper)"
+      gripper_joint_name="$(arg gripper_joint_name)"
+      gripper_max_velocity="$(arg gripper_max_velocity)"
+      gripper_max_force="$(arg gripper_max_force)" >
       <origin xyz="0 0 0.0" rpy="0 0 0" />
     </xacro:load_robot>
