Commit message: sim and mock selection fixed with xacro arg simplification

File: src/kinova_gen3_mock/description/arms/gen3/7dof/urdf/gen3_macro.xacro (robot description, xacro)
@@ -9,5 +9,5 @@
     dof:=7
     vision:=true
-    use_fake_hardware:=false
+    hardware_interface:=mock
     fake_sensor_commands:=false
     mujoco_model:=description/mujoco/scene.xml
@@ -33,5 +33,5 @@
     <xacro:kortex_ros2_control
       name="${prefix}KortexMultiInterfaceHardware" prefix="${prefix}"
-      use_fake_hardware="${use_fake_hardware}"
+      hardware_interface="${hardware_interface}"
       fake_sensor_commands="${fake_sensor_commands}"
       mujoco_model="${mujoco_model}"

File: src/kinova_gen3_mock/description/arms/gen3/7dof/urdf/kortex.ros2_control.xacro (robot description, xacro)
@@ -4,5 +4,5 @@
     name
     prefix
-    use_fake_hardware:=false
+    hardware_interface:=mock
     fake_sensor_commands:=false
     mujoco_model:=description/mujoco/scene.xml
@@ -26,35 +26,33 @@
     <ros2_control name="${name}" type="system">
       <hardware>
-        <xacro:if value="${use_fake_hardware}">
+        <xacro:if value="${hardware_interface == 'mock'}">
           <plugin>mock_components/GenericSystem</plugin>
           <param name="fake_sensor_commands">${fake_sensor_commands}</param>
           <param name="state_following_offset">0.0</param>
         </xacro:if>
-        <xacro:unless value="${use_fake_hardware}">
-          <xacro:if value="${robot_ip != '' and robot_ip != '0.0.0.0'}">
-            <plugin>kortex_driver/KortexMultiInterfaceHardware</plugin>
-            <param name="robot_ip">${robot_ip}</param>
-            <param name="username">${username}</param>
-            <param name="password">${password}</param>
-            <param name="port">${port}</param>
-            <param name="port_realtime">${port_realtime}</param>
-            <param name="session_inactivity_timeout_ms">${session_inactivity_timeout_ms}</param>
-            <param name="connection_inactivity_timeout_ms">${connection_inactivity_timeout_ms}</param>
-            <param name="tf_prefix">"${tf_prefix}"</param>
-            <param name="use_internal_bus_gripper_comm">${use_internal_bus_gripper_comm}</param>
-            <param name="gripper_joint_name">${gripper_joint_name}</param>
-            <param name="gripper_max_velocity">${gripper_max_velocity}</param>
-            <param name="gripper_max_force">${gripper_max_force}</param>
-          </xacro:if>
-          <xacro:unless value="${robot_ip != '' and robot_ip != '0.0.0.0'}">
-            <plugin>picknik_mujoco_ros/MujocoSystem</plugin>
-            <param name="mujoco_model">${mujoco_model}</param>
-            <param name="mujoco_model_package">${mujoco_model_package}</param>
-            <param name="mujoco_viewer">${mujoco_viewer}</param>
-            <param name="mujoco_keyframe">${mujoco_keyframe}</param>
-            <param name="render_publish_rate">10</param>
-            <param name="tf_publish_rate">60</param>
-          </xacro:unless>
-        </xacro:unless>
+        <xacro:if value="${hardware_interface == 'kortex'}">
+          <plugin>kortex_driver/KortexMultiInterfaceHardware</plugin>
+          <param name="robot_ip">${robot_ip}</param>
+          <param name="username">${username}</param>
+          <param name="password">${password}</param>
+          <param name="port">${port}</param>
+          <param name="port_realtime">${port_realtime}</param>
+          <param name="session_inactivity_timeout_ms">${session_inactivity_timeout_ms}</param>
+          <param name="connection_inactivity_timeout_ms">${connection_inactivity_timeout_ms}</param>
+          <param name="tf_prefix">"${tf_prefix}"</param>
+          <param name="use_internal_bus_gripper_comm">${use_internal_bus_gripper_comm}</param>
+          <param name="gripper_joint_name">${gripper_joint_name}</param>
+          <param name="gripper_max_velocity">${gripper_max_velocity}</param>
+          <param name="gripper_max_force">${gripper_max_force}</param>
+        </xacro:if>
+        <xacro:if value="${hardware_interface == 'mujoco'}">
+          <plugin>picknik_mujoco_ros/MujocoSystem</plugin>
+          <param name="mujoco_model">${mujoco_model}</param>
+          <param name="mujoco_model_package">${mujoco_model_package}</param>
+          <param name="mujoco_viewer">${mujoco_viewer}</param>
+          <param name="mujoco_keyframe">${mujoco_keyframe}</param>
+          <param name="render_publish_rate">10</param>
+          <param name="tf_publish_rate">60</param>
+        </xacro:if>
       </hardware>
       <joint name="${prefix}joint_1">
@@ -135,18 +133,12 @@
         <state_interface name="effort"/>
       </joint>
-      <xacro:unless value="${use_fake_hardware}">
-        <xacro:if value="${robot_ip != '' and robot_ip != '0.0.0.0'}">
-          <xacro:unless value="${not gripper}">
-            <xacro:if value="${use_internal_bus_gripper_comm}">
-              <joint name="${prefix}${gripper_joint_name}">
-                <command_interface name="position" />
-                <state_interface name="position"/>
-                <state_interface name="velocity"/>
-              </joint>
-            </xacro:if>
-          </xacro:unless>
-        </xacro:if>
-      </xacro:unless>
-      <xacro:if value="${use_fake_hardware or robot_ip == '' or robot_ip == '0.0.0.0'}">
+      <xacro:if value="${hardware_interface == 'kortex' and gripper and use_internal_bus_gripper_comm}">
+        <joint name="${prefix}${gripper_joint_name}">
+          <command_interface name="position" />
+          <state_interface name="position"/>
+          <state_interface name="velocity"/>
+        </joint>
+      </xacro:if>
+      <xacro:if value="${hardware_interface == 'mock' or hardware_interface == 'mujoco'}">
         <!-- These state values are set for mock and MuJoCo teleoperation with the VFC. -->
         <sensor name="fts">

File: src/kinova_gen3_mock/description/grippers/robotiq_2f_85/urdf/robotiq_2f_85_macro.xacro (robot description, xacro)
@@ -4,5 +4,5 @@
     parent
     prefix
-    use_fake_hardware:=false
+    hardware_interface:=mock
     use_internal_bus_gripper_comm:=false
     fake_sensor_commands:=false">
@@ -14,5 +14,5 @@
         include_ros2_control="${not use_internal_bus_gripper_comm}"
         com_port="/dev/ttyUSB0"
-        use_fake_hardware="${use_fake_hardware}"
+        use_fake_hardware="${hardware_interface != 'kortex'}"
         fake_sensor_commands="${fake_sensor_commands}">
         <origin xyz="0 0 0" rpy="0 0 0" />

File: src/kinova_gen3_mock/description/kortex_robot.xacro (robot description, xacro)
@@ -6,5 +6,5 @@
     prefix:=''
     vision:=true
-    use_fake_hardware:=false
+    hardware_interface:=mock
     fake_sensor_commands:=false
     mujoco_model:=description/mujoco/scene.xml
@@ -33,5 +33,5 @@
       vision="${vision}"
       prefix="${prefix}"
-      use_fake_hardware="${use_fake_hardware}"
+      hardware_interface="${hardware_interface}"
       fake_sensor_commands="${fake_sensor_commands}"
       mujoco_model="${mujoco_model}"
@@ -60,5 +60,5 @@
       parent="${prefix}${last_arm_link}"
       prefix="${prefix}"
-      use_fake_hardware="${use_fake_hardware}"
+      hardware_interface="${hardware_interface}"
       use_internal_bus_gripper_comm="${use_internal_bus_gripper_comm}"
       fake_sensor_commands="${fake_sensor_commands}"/>

File: src/kinova_gen3_mock/description/picknik_kinova_gen3.xacro (robot description, xacro)
@@ -4,5 +4,5 @@
     <xacro:arg name="prefix" default="" />
     <xacro:arg name="vision" default="true" />
-    <xacro:arg name="use_fake_hardware" default="false" />
+    <xacro:arg name="hardware_interface" default="mock" />
     <xacro:arg name="fake_sensor_commands" default="false" />
     <xacro:arg name="mujoco_model" default="description/mujoco/scene.xml" />
@@ -37,5 +37,5 @@
       prefix="$(arg prefix)"
       vision="$(arg vision)"
-      use_fake_hardware="$(arg use_fake_hardware)"
+      hardware_interface="$(arg hardware_interface)"
       fake_sensor_commands="$(arg fake_sensor_commands)"
       mujoco_model="$(arg mujoco_model)"
